Commit message: change box size

File: ros2_grasping/urdf/blue_box.urdf (robot description, URDF)
Before this commit: robot blue_box, 1 links, 0 joints
Links:
- link blue_box: geometry collision box size=0.04 0.04 0.04; visual box size=0.04 0.04 0.04

File: ros2_grasping/urdf/green_box.urdf (robot description, URDF)
Before this commit: robot green_box, 1 links, 0 joints
Links:
- link green_box: geometry collision box size=0.04 0.04 0.04; visual box size=0.04 0.04 0.04

File: ros2_grasping/urdf/red_box.urdf (robot description, URDF)
Before this commit: robot red_box, 1 links, 0 joints
Links:
- link red_box: geometry collision box size=0.04 0.04 0.04; visual box size=0.04 0.04 0.04
