Commit message: use panda robot

File: PandaRobot/panda_ros2_gazebo/urdf/panda.urdf.xacro (robot description, xacro)
@@ -84,5 +84,5 @@
         <origin xyz="0 0 0" rpy=" 0 0 0"/>
         <geometry>
-          <box size = "0.2 0.2 1.3"/>
+          <box size = "0.2 0.2 0.5"/>
         </geometry>
       </collision>
@@ -90,5 +90,5 @@
         <origin xyz="0 0 0" rpy=" 0 0 0"/>
         <geometry>
-          <box size = "0.2 0.2 1.3"/>
+          <box size = "0.2 0.2 0.5"/>
         </geometry>
         <material name="red">
@@ -103,11 +103,102 @@
       <parent link="world" />
       <child link = "panda_base" />
-      <origin xyz="0.0 0.0 0.65" rpy="0.0 0.0 0.0" />
+      <origin xyz="0.0 0.0 0.25" rpy="0.0 0.0 0.0" />
     </joint>
     <joint name="panda_joint" type="fixed">
       <parent link="panda_base" />
       <child link = "panda_link0" />
-      <origin xyz="0.0 0.0 0.655" rpy="0.0 0.0 0.0" />
-    </joint>
+      <origin xyz="0.0 0.0 0.255" rpy="0.0 0.0 0.0" />
+    </joint>
+    <link name='table'>
+      <inertial>
+        <origin xyz="0 0 0" rpy="0 0 0"/>
+        <mass value="100"/>
+        <inertia ixx="0.01"  ixy="0"  ixz="0" iyy="0.01" iyz="0" izz="0.01" />
+      </inertial>
+      <collision name='collision'>
+        <origin xyz="0 0 0" rpy=" 0 0 0"/>
+        <geometry>
+          <box size = "0.5 1.0 0.7"/>
+        </geometry>
+      </collision>
+      <visual name='chassis_visual'>
+        <origin xyz="0 0 0" rpy=" 0 0 0"/>
+        <geometry>
+          <box size = "0.5 1.0 0.7"/>
+        </geometry>
+        <material name="black">
+          <color rgba="1 0 0 1"/>
+        </material>
+      </visual>
+    </link>
+    <joint name="table_world" type="fixed">
+      <parent link="world" />
+      <child link = "table" />
+      <origin xyz="0.5 0.0 0.35" rpy="0.0 0.0 0.0" />
+    </joint>
+    <!-- CAMERA ELEMENTS -->
+    <xacro:property name="camera_link" value="0.05" /> <!-- Size of square 'camera' box -->
+    <!-- Camera link -->
+    <link name="camera_link">
+      <collision>
+        <origin xyz="0 0 0" rpy="0 0 0"/>
+        <geometry>
+          <box size="${camera_link} ${camera_link} ${camera_link}"/>
+        </geometry>
+      </collision>
+      <visual>
+        <origin xyz="0 0 0" rpy="0 0 0"/>
+        <geometry>
+          <box size="${camera_link} ${camera_link} ${camera_link}"/>
+        </geometry>
+        <material name="red"/>
+      </visual>
+      <inertial>
+        <mass value="1e-5" />
+        <origin xyz="0 0 0" rpy="0 0 0"/>
+        <inertia ixx="1e-6" ixy="0" ixz="0" iyy="1e-6" iyz="0" izz="1e-6" />
+      </inertial>
+    </link>
+    <gazebo reference="camera_link">
+      <material>Gazebo/Green</material>
+    </gazebo>
+    <!-- Camera joint (over the center of the table) -->
+    <joint name="camera_joint" type="fixed">
+      <parent link="world" />
+      <child link="camera_link" />
+      <origin xyz="0.5 0 1.35" rpy="0 1.57079632679 0"/>
+    </joint>
+    <!-- Camera sensor -->
+    <gazebo reference="camera_link">
+      <sensor type="camera" name="camera1">
+        <update_rate>10.0</update_rate>
+        <camera name="head">
+          <horizontal_fov>1.3962634</horizontal_fov>
+          <image>
+            <width>800</width>
+            <height>400</height>
+            <format>R8G8B8</format>
+          </image>
+          <clip>
+            <near>0.02</near>
+            <far>300</far>
+          </clip>
+        </camera>
+        <plugin name="camera_controller" filename="libgazebo_ros_camera.so">
+          <alwaysOn>true</alwaysOn>
+          <updateRate>0.0</updateRate>
+          <cameraName>/camera1</cameraName>
+          <imageTopicName>image_raw</imageTopicName>
+          <cameraInfoTopicName>camera_info</cameraInfoTopicName>
+          <frameName>camera_link</frameName>
+          <hackBaseline>0.07</hackBaseline>
+          <distortionK1>0.0</distortionK1>
+          <distortionK2>0.0</distortionK2>
+          <distortionK3>0.0</distortionK3>
+          <distortionT1>0.0</distortionT1>
+          <distortionT2>0.0</distortionT2>
+        </plugin>
+      </sensor>
+    </gazebo>
   </xacro:if>
 </robot>

Commit message: fix inertia of objects

File: PandaRobot/panda_ros2_gazebo/urdf/panda.urdf.xacro (robot description, xacro)
@@ -114,5 +114,5 @@
         <origin xyz="0 0 0" rpy="0 0 0"/>
         <mass value="100"/>
-        <inertia ixx="0.01"  ixy="0"  ixz="0" iyy="0.01" iyz="0" izz="0.01" />
+        <inertia ixx="12.41666667"  ixy="0"  ixz="0" iyy="6.16666667" iyz="0" izz="10.41666667" />
       </inertial>
       <collision name='collision'>
